Commit message: modified:   install/rby1_description/share/rby1_description/rviz/robot.rviz 	modified:   src/rby1_description/urdf/rby1a/model_v1.0.urdf 	modified:   src/rby1_description/urdf/rby1a/model_v1.1.urdf

File: src/rby1_description/urdf/rby1a/model_v1.0.urdf (robot description, URDF)
Before this commit: robot RBY1_A_v1_0, 34 links, 33 joints
Links:
- added link ee_virtual_left, mass 0.0; visual box size=0.0 0.0 0.0
- added link ee_virtual_right, mass 0.0; visual box size=0.0 0.0 0.0
Joints:
- added joint end_effector_left: type fixed, parent link_left_arm_6, child ee_virtual_left, origin xyz=0.0 0.0 -0.1087 rpy=0.0 0.0 0.0, axis 0 0 1
- added joint end_effector_right: type fixed, parent link_right_arm_6, child ee_virtual_right, origin xyz=0.0 0.0 -0.1087 rpy=0.0 0.0 0.0, axis 0 0 1
- joint tool_left: origin xyz=0.0 0.0 -0.1087 rpy=0.0 0.0 0 -> xyz=0.0 0.0 0.0 rpy=0.0 0.0 0; parent link_left_arm_6 -> ee_virtual_left
- joint tool_right: origin xyz=0.0 0.0 -0.1087 rpy=0.0 0.0 0.0 -> xyz=0.0 0.0 0.0 rpy=0.0 0.0 0.0; parent link_right_arm_6 -> ee_virtual_right

File: src/rby1_description/urdf/rby1a/model_v1.1.urdf (robot description, URDF)
Before this commit: robot RBY1_A_v1_1, 34 links, 33 joints
Joints:
- joint tool_left: origin xyz=0.0 0.0 -0.1261 rpy=0.0 0.0 0 -> xyz=0.0 0.0 0.0 rpy=0.0 0.0 0; parent link_left_arm_6 -> ee_virtual_left
- joint tool_right: origin xyz=0.0 0.0 -0.1261 rpy=0.0 0.0 0.0 -> xyz=0.0 0.0 0.0 rpy=0.0 0.0 0.0; parent link_right_arm_6 -> ee_virtual_right

Commit message: modified:   src/rby1_description/urdf/rby1a/model_v1.0.urdf 	modified:   src/rby1_description/urdf/rby1a/model_v1.2.urdf

File: src/rby1_description/urdf/rby1a/model_v1.0.urdf (robot description, URDF)
Before this commit: robot RBY1_A_v1_0, 36 links, 35 joints
Joints:
- joint gripper_finger_l2: axis 1 0 0 -> -1 0 0; mimic (none) -> joint=gripper_finger_l1 multiplier=1.0 offset=0.0
- joint gripper_finger_r2: axis 1 0 0 -> -1 0 0; mimic (none) -> joint=gripper_finger_r1 multiplier=1.0 offset=0.0

File: src/rby1_description/urdf/rby1a/model_v1.2.urdf (robot description, URDF)
Before this commit: robot RBY1_A_v1_2, 32 links, 31 joints
Links:
- added link ee_virtual_left, mass 0.0; visual box size=0.0 0.0 0.0
- added link ee_virtual_right, mass 0.0; visual box size=0.0 0.0 0.0
Joints:
- added joint end_effector_left: type fixed, parent link_left_arm_6, child ee_virtual_left, origin xyz=0.0 0.0 -0.1261 rpy=0.0 0.0 0.0, axis 0 0 1
- added joint end_effector_right: type fixed, parent link_right_arm_6, child ee_virtual_right, origin xyz=0.0 0.0 -0.1261 rpy=0.0 0.0 0.0, axis 0 0 1
- joint gripper_finger_l2: axis 1 0 0 -> -1 0 0; mimic (none) -> joint=gripper_finger_l1 multiplier=1.0 offset=0.0
- joint gripper_finger_r2: axis 1 0 0 -> -1 0 0; mimic (none) -> joint=gripper_finger_r1 multiplier=1.0 offset=0.0
- joint tool_left: origin xyz=0.0 0.0 -0.1261 rpy=0.0 0.0 0 -> xyz=0.0 0.0 0.0 rpy=0.0 0.0 0; parent link_left_arm_6 -> ee_virtual_left
- joint tool_right: origin xyz=0.0 0.0 -0.1261 rpy=0.0 0.0 0.0 -> xyz=0.0 0.0 0.0 rpy=0.0 0.0 0.0; parent link_right_arm_6 -> ee_virtual_right
